Commit message: Added new Shunk with updated appearance, actuated chuck and action for open and close and start operation and end operation. Also decoupled shunk controlers from action

File: fetchit_challenge/urdf/shunk_machine.urdf (robot description, URDF)
Before this commit: robot cartpole_v0, 4 links, 3 joints
Links:
- added link lathe_gripper1_link, mass 0.5; collision mesh filename=package://fetchit_challenge/models/shunk_machine/meshes/shu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; visual mesh filename=package://fetchit_challenge/models/shunk_machine/meshes/shu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
- added link lathe_gripper2_link, mass 0.5; collision mesh filename=package://fetchit_challenge/models/shunk_machine/meshes/shu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; visual mesh filename=package://fetchit_challenge/models/shunk_machine/meshes/shu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
- added link lathe_gripper3_link, mass 0.5; collision mesh filename=package://fetchit_challenge/models/shunk_machine/meshes/shu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; visual mesh filename=package://fetchit_challenge/models/shunk_machine/meshes/shu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
- link lathe_link: geometry collision mesh filename=package://fetchit_challenge/models/shunk_machine/meshes/shu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; visual mesh filename=package://fetchit_challenge/models/shunk_machine/meshes/shu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
Joints:
- added joint lathe_gripper1_joint: type prismatic, parent lathe_link, child lathe_gripper1_link, origin xyz=0.072422 0.0932665 0.0 rpy=0 3.1416 0, axis 1 0 0, limit lower=0.0 upper=0.02 effort=100.0 velocity=1.0
- added joint lathe_gripper2_joint: type prismatic, parent lathe_link, child lathe_gripper2_link, origin xyz=-0.036381 0.0932665 0.0635819 rpy=0 1.0472 0, axis 1 0 0, limit lower=0.0 upper=0.02 effort=100.0 velocity=1.0
- added joint lathe_gripper3_joint: type prismatic, parent lathe_link, child lathe_gripper3_link, origin xyz=-0.036381 0.0932665 -0.0635819 rpy=0 -1.0472 0, axis 1 0 0, limit lower=0.0 upper=0.02 effort=100.0 velocity=1.0
